Commit message: add new fvlm server

File: api/src/nicomotion/scripts/nicomotion/urdf/kinematics.urdf (robot description, URDF)
Before this commit: robot complete, 45 links, 44 joints
Links:
- link finger_segment:11: geometry collision mesh filename=meshes/finger_segment_ipt_50d2a7f4.STL scale=0.001 0.001 0.001; visual mesh filename=meshes/finger_segment_ipt_50d2a7f4.STL scale=0.001 0.001 0.001
- link finger_segment:12: geometry collision mesh filename=meshes/finger_segment_ipt_50d2a7f4.STL scale=0.001 0.001 0.001; visual mesh filename=meshes/finger_segment_ipt_50d2a7f4.STL scale=0.001 0.001 0.001
- link finger_segment:13: geometry collision mesh filename=meshes/finger_segment_ipt_50d2a7f4.STL scale=0.001 0.001 0.001; visual mesh filename=meshes/finger_segment_ipt_50d2a7f4.STL scale=0.001 0.001 0.001
- link finger_segment:14: geometry collision mesh filename=meshes/finger_segment_ipt_50d2a7f4.STL scale=0.001 0.001 0.001; visual mesh filename=meshes/finger_segment_ipt_50d2a7f4.STL scale=0.001 0.001 0.001
- link finger_segment:15: geometry collision mesh filename=meshes/finger_segment_ipt_50d2a7f4.STL scale=0.001 0.001 0.001; visual mesh filename=meshes/finger_segment_ipt_50d2a7f4.STL scale=0.001 0.001 0.001
- link finger_segment:16: geometry collision mesh filename=meshes/finger_segment_ipt_50d2a7f4.STL scale=0.001 0.001 0.001; visual mesh filename=meshes/finger_segment_ipt_50d2a7f4.STL scale=0.001 0.001 0.001
- link finger_segment:21: geometry collision mesh filename=meshes/finger_segment_ipt_50d2a7f4.STL scale=0.001 0.001 0.001; visual mesh filename=meshes/finger_segment_ipt_50d2a7f4.STL scale=0.001 0.001 0.001
- link finger_segment:22: geometry collision mesh filename=meshes/finger_segment_ipt_50d2a7f4.STL scale=0.001 0.001 0.001; visual mesh filename=meshes/finger_segment_ipt_50d2a7f4.STL scale=0.001 0.001 0.001
- link finger_segment:23: geometry collision mesh filename=meshes/finger_segment_ipt_50d2a7f4.STL scale=0.001 0.001 0.001; visual mesh filename=meshes/finger_segment_ipt_50d2a7f4.STL scale=0.001 0.001 0.001
- link finger_segment:24: geometry collision mesh filename=meshes/finger_segment_ipt_50d2a7f4.STL scale=0.001 0.001 0.001; visual mesh filename=meshes/finger_segment_ipt_50d2a7f4.STL scale=0.001 0.001 0.001
- link finger_segment:25: geometry collision mesh filename=meshes/finger_segment_ipt_50d2a7f4.STL scale=0.001 0.001 0.001; visual mesh filename=meshes/finger_segment_ipt_50d2a7f4.STL scale=0.001 0.001 0.001
- link finger_segment:26: geometry collision mesh filename=meshes/finger_segment_ipt_50d2a7f4.STL scale=0.001 0.001 0.001; visual mesh filename=meshes/finger_segment_ipt_50d2a7f4.STL scale=0.001 0.001 0.001
- link fingertip:11: geometry collision mesh filename=meshes/fingertip_ipt_8417b8a9.STL scale=0.001 0.001 0.001; visual mesh filename=meshes/fingertip_ipt_8417b8a9.STL scale=0.001 0.001 0.001
- link fingertip:12: geometry collision mesh filename=meshes/fingertip_ipt_8417b8a9.STL scale=0.001 0.001 0.001; visual mesh filename=meshes/fingertip_ipt_8417b8a9.STL scale=0.001 0.001 0.001
- link fingertip:13: geometry collision mesh filename=meshes/fingertip_ipt_8417b8a9.STL scale=0.001 0.001 0.001; visual mesh filename=meshes/fingertip_ipt_8417b8a9.STL scale=0.001 0.001 0.001
- link fingertip:14: geometry collision mesh filename=meshes/fingertip_ipt_8417b8a9.STL scale=0.001 0.001 0.001; visual mesh filename=meshes/fingertip_ipt_8417b8a9.STL scale=0.001 0.001 0.001
- link fingertip:15: geometry collision mesh filename=meshes/fingertip_ipt_8417b8a9.STL scale=0.001 0.001 0.001; visual mesh filename=meshes/fingertip_ipt_8417b8a9.STL scale=0.001 0.001 0.001
- link fingertip:16: geometry collision mesh filename=meshes/fingertip_ipt_8417b8a9.STL scale=0.001 0.001 0.001; visual mesh filename=meshes/fingertip_ipt_8417b8a9.STL scale=0.001 0.001 0.001
- link head:21: geometry collision mesh filename=meshes/head_iam_b9cf2ea.STL scale=0.001 0.001 0.001; visual mesh filename=meshes/head_iam_b9cf2ea.STL scale=0.001 0.001 0.001
- link left_ankle:11: geometry collision mesh filename=meshes/right_ankle_MIR_iam_c5a384f4.STL scale=0.001 0.001 0.001; visual mesh filename=meshes/right_ankle_MIR_iam_c5a384f4.STL scale=0.001 0.001 0.001
- link left_collarbone:11: geometry collision mesh filename=meshes/left_upper_arm_iam_49d50008.STL scale=0.001 0.001 0.001; visual mesh filename=meshes/left_upper_arm_iam_49d50008.STL scale=0.001 0.001 0.001
- link left_foot:11: geometry collision mesh filename=meshes/left_foot_iam_620666ef.STL scale=0.001 0.001 0.001; visual mesh filename=meshes/left_foot_iam_620666ef.STL scale=0.001 0.001 0.001
- link left_hip_low:11: geometry collision mesh filename=meshes/right_hip_up2_MIR_iam_b8a74a0a.STL scale=0.001 0.001 0.001; visual mesh filename=meshes/right_hip_up2_MIR_iam_b8a74a0a.STL scale=0.001 0.001 0.001
- link left_hip_up:11: geometry collision mesh filename=meshes/right_hip_up_MIR_iam_386ac7b2.STL scale=0.001 0.001 0.001; visual mesh filename=meshes/right_hip_up_MIR_iam_386ac7b2.STL scale=0.001 0.001 0.001
- link left_lower_arm:11: geometry collision mesh filename=meshes/right_wrist_MIR_iam_dcfe6de3.STL scale=0.001 0.001 0.001; visual mesh filename=meshes/right_wrist_MIR_iam_dcfe6de3.STL scale=0.001 0.001 0.001
- link left_palm:11: geometry collision mesh filename=meshes/left_palm_iam_b92c61b5.STL scale=0.001 0.001 0.001; visual mesh filename=meshes/left_palm_iam_b92c61b5.STL scale=0.001 0.001 0.001
- link left_shank:11: geometry collision mesh filename=meshes/right_shank_MIR_iam_a2a9b5d0.STL scale=0.001 0.001 0.001; visual mesh filename=meshes/right_shank_MIR_iam_a2a9b5d0.STL scale=0.001 0.001 0.001
- link left_shoulder:11: geometry collision mesh filename=meshes/left_shoulder_up_iam_1ca4d925.STL scale=0.001 0.001 0.001; visual mesh filename=meshes/left_shoulder_up_iam_1ca4d925.STL scale=0.001 0.001 0.001
- link left_thigh:11: geometry collision mesh filename=meshes/Thigh_left_complete_iam_5a6ba909.STL scale=0.001 0.001 0.001; visual mesh filename=meshes/Thigh_left_complete_iam_5a6ba909.STL scale=0.001 0.001 0.001
- link left_upper_arm:11: geometry collision mesh filename=meshes/left_lower_arm_iam_5be2a521.STL scale=0.001 0.001 0.001; visual mesh filename=meshes/left_lower_arm_iam_5be2a521.STL scale=0.001 0.001 0.001
- link left_wrist:11: geometry collision mesh filename=meshes/left_wrist_iam_c75e4b6f.STL scale=0.001 0.001 0.001; visual mesh filename=meshes/left_wrist_iam_c75e4b6f.STL scale=0.001 0.001 0.001
- link neck:11: geometry collision mesh filename=meshes/neck_iam_61141f4f.STL scale=0.001 0.001 0.001; visual mesh filename=meshes/neck_iam_61141f4f.STL scale=0.001 0.001 0.001
- link right_ankle:11: geometry collision mesh filename=meshes/right_ankle_iam_f4f7d16a.STL scale=0.001 0.001 0.001; visual mesh filename=meshes/right_ankle_iam_f4f7d16a.STL scale=0.001 0.001 0.001
- link right_collarbone:11: geometry collision mesh filename=meshes/right_upper_arm_iam_e3e9c979.STL scale=0.001 0.001 0.001; visual mesh filename=meshes/right_upper_arm_iam_e3e9c979.STL scale=0.001 0.001 0.001
- link right_foot:11: geometry collision mesh filename=meshes/right_foot_iam_3ff7356a.STL scale=0.001 0.001 0.001; visual mesh filename=meshes/right_foot_iam_3ff7356a.STL scale=0.001 0.001 0.001
- link right_hip_low:11: geometry collision mesh filename=meshes/right_hip_up2_iam_f4f7d16a.STL scale=0.001 0.001 0.001; visual mesh filename=meshes/right_hip_up2_iam_f4f7d16a.STL scale=0.001 0.001 0.001
- link right_hip_up:11: geometry collision mesh filename=meshes/right_hip_up_iam_f46f7684.STL scale=0.001 0.001 0.001; visual mesh filename=meshes/right_hip_up_iam_f46f7684.STL scale=0.001 0.001 0.001
- link right_lower_arm:11: geometry collision mesh filename=meshes/right_wrist_iam_771ea33e.STL scale=0.001 0.001 0.001; visual mesh filename=meshes/right_wrist_iam_771ea33e.STL scale=0.001 0.001 0.001
- link right_palm:11: geometry collision mesh filename=meshes/right_palm_iam_583b22df.STL scale=0.001 0.001 0.001; visual mesh filename=meshes/right_palm_iam_583b22df.STL scale=0.001 0.001 0.001
- link right_shank:11: geometry collision mesh filename=meshes/right_shank_iam_7a73fe91.STL scale=0.001 0.001 0.001; visual mesh filename=meshes/right_shank_iam_7a73fe91.STL scale=0.001 0.001 0.001
- link right_shoulder:11: geometry collision mesh filename=meshes/right_shoulder_up_iam_34db21c8.STL scale=0.001 0.001 0.001; visual mesh filename=meshes/right_shoulder_up_iam_34db21c8.STL scale=0.001 0.001 0.001
- link right_thigh:11: geometry collision mesh filename=meshes/Thigh_right_complete_iam_6502f197.STL scale=0.001 0.001 0.001; visual mesh filename=meshes/Thigh_right_complete_iam_6502f197.STL scale=0.001 0.001 0.001
- link right_upper_arm:11: geometry collision mesh filename=meshes/right_lower_arm1_iam_65a34910.STL scale=0.001 0.001 0.001; visual mesh filename=meshes/right_lower_arm1_iam_65a34910.STL scale=0.001 0.001 0.001
- link right_wrist:11: geometry collision mesh filename=meshes/right_wrist_iam_81504746.STL scale=0.001 0.001 0.001; visual mesh filename=meshes/right_wrist_iam_81504746.STL scale=0.001 0.001 0.001
- link torso:11: geometry collision mesh filename=meshes/torso_iam_fb80b350.STL scale=0.001 0.001 0.001; visual mesh filename=meshes/torso_iam_fb80b350.STL scale=0.001 0.001 0.001
